Commit message: odom

File: description/robot_core.xacro (robot description, xacro)
@@ -10,5 +10,5 @@
     <xacro:property name="wheel_mass" value="0.1"/>
     <xacro:property name="wheel_offset_x" value="0.155"/>
-    <xacro:property name="wheel_offset_y" value="0.0975"/>
+    <xacro:property name="wheel_offset_y" value="0.085"/>
     <xacro:property name="wheel_offset_z" value="-0.02"/>
     <xacro:property name="caster_wheel_radius" value="0.01"/>

File: description/ros2_control.xacro (robot description, xacro)
@@ -10,5 +10,5 @@
             <param name="baud_rate">57600</param>
             <param name="timeout">1000</param>
-            <param name="enc_counts_per_rev">3294</param>
+            <param name="enc_counts_per_rev">3270</param>
         </hardware>
         <joint name="left_wheel_joint">
